Commit message: SLAM work untuk simulnya wkwk

File: urdf/robot.urdf.xacro (robot description, xacro)
@@ -1,5 +1,4 @@
 <?xml version="1.0"?>
 <robot name="robot" xmlns:xacro="http://www.ros.org/wiki/xacro">
-  <!-- Parameter ukuran robot -->
   <xacro:property name="base_length"  value="0.20"/>
   <xacro:property name="base_width"   value="0.15"/>
@@ -7,12 +6,12 @@
   <xacro:property name="wheel_radius" value="0.033"/>
   <xacro:property name="wheel_width"  value="0.02"/>
-  <xacro:property name="track_width"  value="0.15"/>   <!-- jarak kiri-kanan -->
-  <xacro:property name="wheel_xoff"   value="0.07"/>   <!-- jarak depan-belakang dari center -->
-  <!-- Macro roda agar tidak copy-paste -->
+  <xacro:property name="track_width"  value="0.15"/>
+  <xacro:property name="wheel_xoff"   value="0.07"/>
+  <!-- Macro roda: hanya definisi joint + link + friction dasar -->
   <xacro:macro name="wheel" params="name x y">
     <joint name="${name}_joint" type="continuous">
       <parent link="base_link"/>
       <child  link="${name}"/>
-      <origin xyz="${x} ${y} 0" rpy="-1.5708 0 0"/>
+      <origin xyz="${x} ${y} ${-base_height/2}" rpy="-1.5708 0 0"/>
       <axis xyz="0 0 1"/>
       <dynamics damping="0.1" friction="0.1"/>
@@ -38,11 +37,4 @@
       </inertial>
     </link>
-    <!-- Friction tinggi agar tidak slip -->
-    <gazebo reference="${name}">
-      <mu1>1.0</mu1>
-      <mu2>1.0</mu2>
-      <kp>1000000.0</kp>
-      <kd>1.0</kd>
-    </gazebo>
   </xacro:macro>
   <!-- ── Base link ──────────────────────────────────────── -->
@@ -51,6 +43,5 @@
     <parent link="base_footprint"/>
     <child  link="base_link"/>
-    <!-- Z tepat setinggi jari-jari roda agar roda menyentuh ground -->
-    <origin xyz="0 0 ${wheel_radius}" rpy="0 0 0"/>
+    <origin xyz="0 0 ${wheel_radius + base_height/2}" rpy="0 0 0"/>
   </joint>
   <link name="base_link">
@@ -70,5 +61,4 @@
     <inertial>
       <mass value="1.0"/>
-      <!-- Inertia box: I = m/12 * (a²+b²) -->
       <inertia ixx="0.00347" iyy="0.00413" izz="0.00680"
                ixy="0"       ixz="0"       iyz="0"/>
@@ -76,14 +66,38 @@
   </link>
   <!-- ── 4 Roda ─────────────────────────────────────────── -->
-  <!--        nama            x              y            -->
-  <xacro:wheel name="front_left"  x=" ${wheel_xoff}"  y=" ${track_width/2}"/>
-  <xacro:wheel name="front_right" x=" ${wheel_xoff}"  y="-${track_width/2}"/>
-  <xacro:wheel name="rear_left"   x="-${wheel_xoff}"  y=" ${track_width/2}"/>
-  <xacro:wheel name="rear_right"  x="-${wheel_xoff}"  y="-${track_width/2}"/>
+  <xacro:wheel name="front_left"  x=" ${wheel_xoff}" y=" ${track_width/2}"/>
+  <xacro:wheel name="front_right" x=" ${wheel_xoff}" y="-${track_width/2}"/>
+  <xacro:wheel name="rear_left"   x="-${wheel_xoff}" y=" ${track_width/2}"/>
+  <xacro:wheel name="rear_right"  x="-${wheel_xoff}" y="-${track_width/2}"/>
+  <!-- Friction roda depan: grip tinggi (penggerak) -->
+  <gazebo reference="front_left">
+    <mu1>1.0</mu1>
+    <mu2>1.0</mu2>
+    <kp>1000000.0</kp>
+    <kd>1.0</kd>
+  </gazebo>
+  <gazebo reference="front_right">
+    <mu1>1.0</mu1>
+    <mu2>1.0</mu2>
+    <kp>1000000.0</kp>
+    <kd>1.0</kd>
+  </gazebo>
+  <!-- Friction roda belakang: rendah agar passive/free rolling -->
+  <gazebo reference="rear_left">
+    <mu1>0.01</mu1>
+    <mu2>0.01</mu2>
+    <kp>100000.0</kp>
+    <kd>1.0</kd>
+  </gazebo>
+  <gazebo reference="rear_right">
+    <mu1>0.01</mu1>
+    <mu2>0.01</mu2>
+    <kp>100000.0</kp>
+    <kd>1.0</kd>
+  </gazebo>
   <!-- ── Laser frame ────────────────────────────────────── -->
   <joint name="laser_joint" type="fixed">
     <parent link="base_link"/>
     <child  link="laser"/>
-    <!-- Tengah atas body, rotasi 0 agar scan simetris -->
     <origin xyz="0.05 0 ${base_height/2 + 0.02}" rpy="0 0 0"/>
   </joint>
@@ -104,14 +118,9 @@
   </link>
   <!-- ── Gazebo plugins ─────────────────────────────────── -->
-  <!-- Diff drive: gunakan roda depan sebagai penggerak utama -->
   <gazebo>
     <plugin filename="libignition-gazebo-diff-drive-system.so"
             name="ignition::gazebo::systems::DiffDrive">
-      <!-- Kiri: depan + belakang dikopel -->
       <left_joint>front_left_joint</left_joint>
-      <left_joint>rear_left_joint</left_joint>
-      <!-- Kanan: depan + belakang dikopel -->
       <right_joint>front_right_joint</right_joint>
-      <right_joint>rear_right_joint</right_joint>
       <wheel_separation>${track_width}</wheel_separation>
       <wheel_radius>${wheel_radius}</wheel_radius>
@@ -128,5 +137,4 @@
     </plugin>
   </gazebo>
-  <!-- Joint state publisher -->
   <gazebo>
     <plugin filename="libignition-gazebo-joint-state-publisher-system.so"
@@ -135,5 +143,4 @@
     </plugin>
   </gazebo>
-  <!-- Laser scanner -->
   <gazebo reference="laser">
     <sensor name="laser_sensor" type="gpu_lidar">
